File: DigiSporc.sch (EAGLE design)
At the start: 12 parts, among them IC0 ATTINY45DIP8, IC1 7805L

Commit message: Schematics and board in .png added
Other:
- note added: "ATtiny45/85 based Arduino Clone"
- note added: "by Marco Losurdo"
- note removed: "Tiny Arduino Clone for ATtiny45/85"
- note removed: "by Marco"
Changed lines of the file:
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@@
 <sheet>
 <plain>
-<text x="119.38" y="-3.81" size="2.286" layer="94">Tiny Arduino Clone for ATtiny45/85</text>
-<text x="119.38" y="-7.62" size="2.286" layer="94">by Marco</text>
+<text x="119.38" y="-3.81" size="2.286" layer="94">ATtiny45/85 based Arduino Clone</text>
+<text x="119.38" y="-7.62" size="2.286" layer="94">by Marco Losurdo</text>
 <text x="119.38" y="-11.43" size="2.286" layer="94">License CC-BY-SA 3.0</text>
 <text x="210.82" y="-27.94" size="2.286" layer="94">1</text>
