File: DigiSporc_nano.brd (EAGLE design)
At the start: 19.7 x 14.3 mm, 8 parts, among them IC0 ATTINY45DIP8

Commit message: Link Update
Aggiornato link ad hardware support per ATtiny.
Routing:
- net GND: track 25.9 -> 0.00 mm, vias 0 -> 1
- net RESET: track 23.0 -> 20.4 mm
- net PIN3: track 12.3 -> 11.0 mm
- net PIN4: track 6.50 -> 5.39 mm
- net PIN2: track 14.1 -> 13.0 mm
- net N$5: track 19.4 -> 18.4 mm
